File: board/board.kicad_pcb (KiCad board)
At the start: 2 copper layers, 96.8 x 80.9 mm, 32 parts, among them J1 RPi_Header, J2 Smoke_Sensor, J3 LEDs, J4 Temp_Sensor, J5 Alarm, J6 Conn_01x03, J7 Fan_Power, J8 USB_Power, J9 Coil, Q1 Q_PMOS_GDS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

Commit message: Added labels
Other:
- board text added: "ALARM"
- board text added: "COIL"
- board text added: "FAN"
- board text added: "LEDs"
- board text added: "SMOKE"
- board text added: "TEMP"
- board text added: "UART"
- board text added: "USB_OUT"
Changed lines of the file:
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@@
-(kicad_pcb (version 20171130) (host pcbnew "(5.0.2)-1")
+(kicad_pcb (version 20171130) (host pcbnew 5.0.2-bee76a0~70~ubuntu18.04.1)
   (general
     (thickness 1.6)
-    (drawings 15)
+    (drawings 23)
     (tracks 165)
     (zones 0)
@@
       (xy 1.126492 -15.143947)) (layer B.SilkS) (width 0.01))
   )
+  (gr_text USB_OUT (at 78.2574 136.1948) (layer F.SilkS)
+    (effects (font (size 1.5 1.5) (thickness 0.3)))
+  )
+  (gr_text ALARM (at 144.399 68.58) (layer F.SilkS)
+    (effects (font (size 1.5 1.5) (thickness 0.3)))
+  )
+  (gr_text LEDs (at 123.1646 70.2056) (layer F.SilkS)
+    (effects (font (size 1.5 1.5) (thickness 0.3)))
+  )
+  (gr_text TEMP (at 96.3676 78.7908) (layer F.SilkS)
+    (effects (font (size 1.5 1.5) (thickness 0.3)))
+  )
+  (gr_text SMOKE (at 82.55 78.6638) (layer F.SilkS)
+    (effects (font (size 1.5 1.5) (thickness 0.3)))
+  )
+  (gr_text FAN (at 139.9794 137.5918) (layer F.SilkS)
+    (effects (font (size 1.5 1.5) (thickness 0.3)))
+  )
+  (gr_text COIL (at 131.9784 137.3632) (layer F.SilkS)
+    (effects (font (size 1.5 1.5) (thickness 0.3)))
+  )
+  (gr_text UART (at 107.95 68.0974) (layer F.SilkS)
+    (effects (font (size 1.5 1.5) (thickness 0.3)))
+  )
   (gr_text v1.0 (at 156.591 142.4686) (layer B.SilkS)
